File: 1 Strain Gauge Board.sch (EAGLE design)
At the start: 39 parts, among them IC1 LM317MABDT, IC2 LM317MABDT, IC3 74LS674DW, J1 SD_CARD_SOCKET, Q1 16MHz, U1 LTC6082HGNPBF, U2 AD5254BRUZ1, U3 MAX11610EEE+, U4 ATMEGA328P_TQFP, U5 TXB0108DQSR

Commit message: Version 1 FINAL
Nearly complete version of the first iteration of the strain gauge logger.
TODO: Check SD card for validity. I have no idea how it's supposed to be hooked up.
Parts:
- removed C1, C2: .1uF, resistor:C-USC1206K
- removed C3: .01uF, resistor:C-USC1206K
- removed C4, C5: 22pF, resistor:C-USC1206K
- removed D1: LED-RGLTST-C195KGJRKT, SparkFun-LED:LED-RGLTST-C195KGJRKT
- removed IC3: 74LS674DW, 74xx-eu:74LS674DW
- removed J1: SD_CARD_SOCKET, SparkFun-Connectors:SD_CARD_SOCKET
- removed Q1: 16MHz, special:XTAL/S
- removed R1, R2: 350, resistor:R-US_M1206
- removed R10: 100k, resistor:R-US_M1206
- removed R11, R5, R6: 10M, resistor:R-US_M1206
- removed R16, R17: 330, resistor:R-US_M1206
- removed R3: 370, resistor:R-US_M1206
- removed R4: 5k, resistor:R-US_M1206
- removed R7: 9.76M, resistor:R-US_M1206
- removed R8: 10K, resistor:R-US_M1206
- removed R9: 100, resistor:R-US_M1206
- removed U1: LTC6082HGNPBF, LTC6082 Strain Gauge Amplifier:LTC6082HGNPBF
- removed U2: AD5254BRUZ1, AD5254 4x1k Digital Potentiometer:AD5254BRUZ1
- removed U3: MAX11610EEE+, MAX11610 10 bit ADC:MAX11610EEE+
- removed U4: ATMEGA328P_TQFP, SparkFun-IC-Microcontroller:ATMEGA328P_TQFP
- removed U5: TXB0108DQSR, SparkFun-IC-Comms:TXB0108
- added -3VSUP: LM317ABDT, v-reg:LM317MABDT
- added -3VSUP-BYP, INPUT-BYP: .1uF, rcl:C-USC1206K
- added -3VSUP-D1: GREEN, SparkFun-LED:LED-GREEN1206
- added -3VSUP-R1: 330, rcl:R-US_M1206
- added -3VSUP-R2: 462, rcl:R-US_M1206
- added -3VSUP-R3: 150, rcl:R-US_M1206
- added 3VSUP-BYP, 5VSUP-BYP: .1uF, resistor:C-USC1206K
- added ADC-1: MAX11610EEE+, MAX11610 10 bit ADC:MAX11610EEE+
- added ADC-BYP, LSHIFT1-BYP-1, LSHIFT1-BYP-2, LSHIFT2-BYP-1, LSHIFT2-BYP-2, POT1-BYP, POT2-BYP, POT3-BYP, SD-BYP, SHREG-BYP: .01uF, resistor:C-USC1206K
- added AMP-1, AMP-2, AMP-3: LTC6082HGNPBFSSOP-16_GN-L, LTC6082 Strain Gauge Amplifier:LTC6082HGNPBFSSOP-16_GN-L
- added AMP1-BYP, AMP2-BYP, AMP3-BYP: .01uF, rcl:C-USC1206K
- added ATMEGA328: ATMEGA328P_TQFP, SparkFun-IC-Microcontroller:ATMEGA328P_TQFP
- added ATMEGA328-BYP: (no value), rcl:C-USC1206
- added CAL-1, CAL-10, CAL-11, CAL-12, CAL-13, CAL-14, CAL-15, CAL-16, CAL-2, CAL-3, CAL-4, CAL-5, CAL-6, CAL-7, CAL-8, CAL-9: LED-RGLTST-C195KGJRKT, SparkFun-LED:LED-RGLTST-C195KGJRKT
- added CAL-1-R1, CAL-1-R2, CAL-10-R1, CAL-10-R2, CAL-11-R1, CAL-11-R2, CAL-12-R1, CAL-12-R2, CAL-13-R1, CAL-13-R2, CAL-14-R1, CAL-14-R2, CAL-15-R1, CAL-15-R2, CAL-16-R1, CAL-16-R2, CAL-2-R1, CAL-2-R2, CAL-3-R1, CAL-3-R2, CAL-4-R1, CAL-4-R2, CAL-5-R1, CAL-5-R2, CAL-6-R1, CAL-6-R2, CAL-7-R1, CAL-7-R2, CAL-8-R1, CAL-8-R2, CAL-9-R1, CAL-9-R2: 330, resistor:R-US_M1206
- added CRYSTAL: 16MHz, special:XTAL/S
- added CRYSTAL-C1, CRYSTAL-C2: 22pF, resistor:C-USC1206K
- added ICSP: (no value), SparkFun-Connectors:CONN_03X2FEMALE
- added LSHIFT-1, LSHIFT-2: TXB0104, SparkFun-IC-Comms:TXB0104PWRSOIC14
- added POT-1, POT-2, POT-3: AD5254BRUZ1, AD5254 4x1k Digital Potentiometer:AD5254BRUZ1
- added POT-WP-R1: 100, rcl:R-US_M1206
- added RESET-PULLUP: 10k, rcl:R-US_M1206
- added SD-SOCKET: SD_CARD_SOCKET, SparkFun-Connectors:SD_CARD_SOCKET
- added SHREG: 74LS674DW, 74xx-eu:74LS674DW
- added WB1-A-C1, WB10-A-C1, WB11-A-C1, WB12-A-C1, WB2-A-C1, WB3-A-C1, WB4-A-C1, WB5-A-C1, WB6-A-C1, WB7-A-C1, WB8-A-C1, WB9-A-C1: 100nF, rcl:C-USC1206K
- added WB1-A-R1, WB1-A-R2, WB10-A-R1, WB10-A-R2, WB11-A-R1, WB11-A-R2, WB12-A-R1, WB12-A-R2, WB2-A-R1, WB2-A-R2, WB3-A-R1, WB3-A-R2, WB4-A-R1, WB4-A-R2, WB5-A-R1, WB5-A-R2, WB6-A-R1, WB6-A-R2, WB7-A-R1, WB7-A-R2, WB8-A-R1, WB8-A-R2, WB9-A-R1, WB9-A-R2: 1k, rcl:R-US_M1206
- added WB1-A-R3, WB1-A-R4, WB10-A-R3, WB10-A-R4, WB11-A-R3, WB11-A-R4, WB12-A-R3, WB12-A-R4, WB2-A-R3, WB2-A-R4, WB3-A-R3, WB3-A-R4, WB4-A-R3, WB4-A-R4, WB5-A-R3, WB5-A-R4, WB6-A-R3, WB6-A-R4, WB7-A-R3, WB7-A-R4, WB8-A-R3, WB8-A-R4, WB9-A-R3, WB9-A-R4: 1M, rcl:R-US_M1206
- added WB1-A-R5, WB10-A-R5, WB11-A-R5, WB12-A-R5, WB2-A-R5, WB3-A-R5, WB4-A-R5, WB5-A-R5, WB6-A-R5, WB7-A-R5, WB8-A-R5, WB9-A-R5: 100k, rcl:R-US_M1206
- added WB1-R1, WB1-R2: 350, resistor:R-US_M1206
- added WB1-R3: 370, resistor:R-US_M1206
- added WB1-R4: 5k, resistor:R-US_M1206
- added WB10-R1, WB10-R2, WB11-R1, WB11-R2, WB12-R1, WB12-R2, WB2-R1, WB2-R2, WB3-R1, WB3-R2, WB4-R1, WB4-R2, WB5-R1, WB5-R2, WB6-R1, WB6-R2, WB7-R1, WB7-R2, WB8-R1, WB8-R2, WB9-R1, WB9-R2: 350, rcl:R-US_M1206
- added WB10-R3, WB11-R3, WB12-R3, WB2-R3, WB3-R3, WB4-R3, WB5-R3, WB6-R3, WB7-R3, WB8-R3, WB9-R3: 370, rcl:R-US_M1206
- added WB10-R4, WB11-R4, WB12-R4, WB2-R4, WB3-R4, WB4-R4, WB5-R4, WB6-R4, WB7-R4, WB8-R4, WB9-R4: 5k, rcl:R-US_M1206
- added X3, X4, X5: (no value), con-phoenix-254:MPT6
- 3VSUP: value LM317MABDT -> LM317ABDT
- renumbered D2 to 5VSUP-D1, D3 to 3VSUP-D1, IC1 to 3VSUP, IC2 to 5VSUP, R12 to 3VSUP-R1, R13 to 3VSUP-R2, R14 to 5VSUP-R1, R15 to 5VSUP-R2, R18 to 3VSUP-R3, R19 to 5VSUP-R3
Connections:
- removed net +3V3: 3VSUP-R1.2, 3VSUP-R3.1, 3VSUP.OUT, C1.2, J1.VDD, R3.2, R4.1, R8.2, U1.V+, U5.VCCA, X1-1.1, X1-4.1, X1-6.1
- removed net N$10: U3.SDA, U4.PC4(ADC4/SDA)
- removed net N$11: U3.SCL, U4.PC5(ADC5/SCL)
- removed net N$16: U4.PD5(T1), U5.OE
- removed net N$3: R11.1, R6.2, U1.-INA
- removed net N$4: R11.2, U1.+INB, U1.OUTA
- removed net N$6: R5.2, R7.1, U1.+INA
- removed net N$7: C2.1, R7.2, R8.1, R9.1
- removed net N$8: C3.2, R10.1, R9.2, U1.-INB
- removed net N$9: C3.1, R10.2, U1.OUTB, U3.AIN0
- new net +3V: 3VSUP-BYP.1, 3VSUP-R1.2, 3VSUP-R3.1, 3VSUP.OUT, AMP-1.V+, AMP-2.V+, AMP-3.V+, AMP1-BYP.2, AMP2-BYP.2, AMP3-BYP.2, LSHIFT-1.VCCA, LSHIFT-2.VCCA, LSHIFT1-BYP-1.1, LSHIFT2-BYP-1.1, POT-1.VDD, POT-2.VDD, POT-3.VDD, POT1-BYP.1, POT2-BYP.1, POT3-BYP.1, SD-BYP.1, SD-SOCKET.VDD, WB1-R3.2, WB1-R4.1, WB10-R3.2, WB10-R4.2, WB11-R3.2, WB11-R4.2, WB12-R3.2, WB12-R4.2, WB2-R3.2, WB2-R4.2, WB3-R3.2, WB3-R4.2, WB4-R3.2, WB4-R4.2, WB5-R3.2, WB5-R4.2, WB6-R3.2, WB6-R4.2, WB7-R3.2, WB7-R4.2, WB8-R3.2, WB8-R4.2, WB9-R3.2, WB9-R4.2, X1-1.1, X1-3.1, X1-5.1, X3-1.1, X3-3.1, X3-5.1, X4-1.1, X4-3.1, X4-5.1, X5-1.1, X5-3.1, X5-5.1
- new net -3V: -3VSUP-R1.2, -3VSUP-R3.1, -3VSUP.OUT
- new net LSHIFT-OE: ATMEGA328.PD5(T1), LSHIFT-1.OE, LSHIFT-2.OE
- new net MISO: ATMEGA328.PB4(MISO), ICSP.1
- new net MOSI: ATMEGA328.PB3(MOSI/OC2), ICSP.4
- new net N$41: CAL-2-R1.2, CAL-2.RC
- new net N$42: CAL-2-R2.2, CAL-2.GC
- new net N$45: CAL-2-R2.1, CAL-2.RA, SHREGA.P1
- new net N$46: CAL-5-R1.2, CAL-5.RC
- new net N$47: CAL-5-R2.2, CAL-5.GC
- new net N$48: CAL-5-R2.1, CAL-5.RA, SHREGA.P4
- new net N$49: CAL-8-R1.2, CAL-8.RC
- new net N$50: CAL-8-R2.2, CAL-8.GC
- new net N$51: CAL-8-R2.1, CAL-8.RA, SHREGA.P7
- new net N$52: CAL-6-R1.2, CAL-6.RC
- new net N$53: CAL-6-R2.2, CAL-6.GC
- new net N$54: CAL-6-R2.1, CAL-6.RA, SHREGA.P5
- new net N$55: CAL-3-R1.2, CAL-3.RC
- new net N$56: CAL-3-R2.2, CAL-3.GC
- new net N$57: CAL-3-R2.1, CAL-3.RA, SHREGA.P2
- new net N$58: CAL-9-R1.2, CAL-9.RC
- new net N$59: CAL-9-R2.2, CAL-9.GC
- new net N$60: CAL-9-R2.1, CAL-9.RA, SHREGA.P8
- new net N$61: CAL-11-R1.2, CAL-11.RC
- new net N$62: CAL-11-R2.2, CAL-11.GC
- new net N$63: CAL-11-R2.1, CAL-11.RA, SHREGA.P10
- new net N$64: CAL-12-R1.2, CAL-12.RC
- new net N$65: CAL-12-R2.2, CAL-12.GC
- new net N$66: CAL-12-R2.1, CAL-12.RA, SHREGA.P11
- new net N$67: CAL-14-R1.2, CAL-14.RC
- new net N$68: CAL-14-R2.2, CAL-14.GC
- new net N$69: CAL-14-R2.1, CAL-14.RA, SHREGA.P13
- new net N$70: CAL-15-R1.2, CAL-15.RC
- new net N$71: CAL-15-R2.2, CAL-15.GC
- new net N$72: CAL-15-R2.1, CAL-15.RA, SHREGA.P14
- new net N$73: CAL-7-R1.2, CAL-7.RC
- new net N$74: CAL-7-R2.2, CAL-7.GC
- new net N$75: CAL-7-R2.1, CAL-7.RA, SHREGA.P6
- new net N$76: CAL-10-R1.2, CAL-10.RC
- new net N$77: CAL-10-R2.2, CAL-10.GC
- new net N$78: CAL-10-R2.1, CAL-10.RA, SHREGA.P9
- new net N$79: CAL-13-R1.2, CAL-13.RC
- new net N$80: CAL-13-R2.2, CAL-13.GC
- new net N$81: CAL-13-R2.1, CAL-13.RA, SHREGA.P12
- new net N$82: CAL-16-R1.2, CAL-16.RC
- new net N$83: CAL-16-R2.2, CAL-16.GC
- new net N$84: CAL-16-R2.1, CAL-16.RA, SHREGA.P15
- new net N$85: CAL-4-R1.2, CAL-4.RC
- new net N$86: CAL-4-R2.2, CAL-4.GC
- new net N$87: CAL-4-R2.1, CAL-4.RA, SHREGA.P3
- new net POT-SELECT-AD0: ATMEGA328.PD3(INT1), POT-1.AD0, POT-2.AD0, POT-3.AD0
- new net POT-SELECT-AD1: ATMEGA328.PD2(INT0), POT-1.AD1, POT-2.AD1, POT-3.AD1
- new net POT-WP: POT-1.!, POT-2.!, POT-3.!, POT-WP-R1.1
- new net RESET: ATMEGA328.PC6(/RESET), ICSP.5, RESET-PULLUP.1
- new net SCK: ATMEGA328.PB5(SCK), ICSP.3
- new net SCL: ADC-1.SCL, ATMEGA328.PC5(ADC5/SCL), POT-1.SCL, POT-2.SCL, POT-3.SCL
- new net SDA: ADC-1.SDA, ATMEGA328.PC4(ADC4/SDA), POT-1.SDA, POT-2.SDA, POT-3.SDA
- new net SG1-AIN: ADC-1.AIN0, WB1-A-C1.1, WB1-A-R5.2
- new net SG1-NEG: WB1-A-R2.1, WB1-R1.2, X1-2.1
- new net SG1-POS: POT-1.B0, WB1-A-R1.1, WB1-R2.2, WB1-R3.1
- new net SG1-POT: POT-1.W0, WB1-R4.2
- new net SG10-AIN: ADC-1.AIN9, WB10-A-C1.1, WB10-A-R5.2
- new net SG10-NEG: WB10-A-R2.1, WB10-R1.2, X5-2.1
- new net SG10-POS: POT-3.B1, WB10-A-R1.1, WB10-R2.2, WB10-R3.1
- new net SG10-POT: POT-3.W1, WB10-R4.1
- new net SG11-AIN: ADC-1.AIN10, WB11-A-C1.1, WB11-A-R5.2
- new net SG11-NEG: WB11-A-R2.1, WB11-R1.2, X5-4.1
- new net SG11-POS: POT-3.B2, WB11-A-R1.1, WB11-R2.2, WB11-R3.1
- new net SG11-POT: POT-3.W2, WB11-R4.1
- new net SG12-AIN: ADC-1.AIN11/REF, WB12-A-C1.1, WB12-A-R5.2
- new net SG12-NEG: WB12-A-R2.1, WB12-R1.2, X5-6.1
- new net SG12-POS: POT-3.B3, WB12-A-R1.1, WB12-R2.2, WB12-R3.1
- new net SG12-POT: POT-3.W3, WB12-R4.1
- new net SG2-AIN: ADC-1.AIN1, WB2-A-C1.1, WB2-A-R5.2
- new net SG2-NEG: WB2-A-R2.1, WB2-R1.2, X1-4.1
- new net SG2-POS: POT-1.B1, WB2-A-R1.1, WB2-R2.2, WB2-R3.1
- new net SG2-POT: POT-1.W1, WB2-R4.1
- new net SG3-AIN: ADC-1.AIN2, WB3-A-C1.1, WB3-A-R5.2
- new net SG3-NEG: WB3-A-R2.1, WB3-R1.2, X1-6.1
- new net SG3-POS: POT-1.B2, WB3-A-R1.1, WB3-R2.2, WB3-R3.1
- new net SG3-POT: POT-1.W2, WB3-R4.1
- new net SG4-AIN: ADC-1.AIN3, WB4-A-C1.1, WB4-A-R5.2
- new net SG4-NEG: WB4-A-R2.1, WB4-R1.2, X3-2.1
- new net SG4-POS: POT-1.B3, WB4-A-R1.1, WB4-R2.2, WB4-R3.1
- new net SG4-POT: POT-1.W3, WB4-R4.1
- new net SG5-AIN: ADC-1.AIN4, WB5-A-C1.1, WB5-A-R5.2
- new net SG5-NEG: WB5-A-R2.1, WB5-R1.2, X3-4.1
- new net SG5-POS: POT-2.B0, WB5-A-R1.1, WB5-R2.2, WB5-R3.1
- new net SG5-POT: POT-2.W0, WB5-R4.1
- new net SG6-AIN: ADC-1.AIN5, WB6-A-C1.1, WB6-A-R5.2
- new net SG6-NEG: WB6-A-R2.1, WB6-R1.2, X3-6.1
- new net SG6-POS: POT-2.B1, WB6-A-R1.1, WB6-R2.2, WB6-R3.1
- new net SG6-POT: POT-2.W1, WB6-R4.1
- new net SG7-AIN: ADC-1.AIN6, WB7-A-C1.1, WB7-A-R5.2
- new net SG7-NEG: WB7-A-R2.1, WB7-R1.2, X4-2.1
- new net SG7-POS: POT-2.B2, WB7-A-R1.1, WB7-R2.2, WB7-R3.1
- new net SG7-POT: POT-2.W2, WB7-R4.1
- new net SG8-AIN: ADC-1.AIN7, WB8-A-C1.1, WB8-A-R5.2
- new net SG8-NEG: WB8-A-R2.1, WB8-R1.2, X4-4.1
- new net SG8-POS: POT-2.B3, WB8-A-R1.1, WB8-R2.2, WB8-R3.1
- new net SG8-POT: POT-2.W3, WB8-R4.1
- new net SG9-AIN: ADC-1.AIN8, WB9-A-C1.1, WB9-A-R5.2
- new net SG9-NEG: WB9-A-R2.1, WB9-R1.2, X4-6.1
- new net SG9-POS: POT-3.B0, WB9-A-R1.1, WB9-R2.2, WB9-R3.1
- new net SG9-POT: POT-3.W0, WB9-R4.1
- new net V-: -3VSUP-BYP.2, -3VSUP-D1.C, -3VSUP-R2.1, AMP-1.V-, AMP-2.V-, AMP-3.V-, AMP1-BYP.1, AMP2-BYP.1, AMP3-BYP.1
- new net WB1-A-NEG: AMP-1.-INA, WB1-A-R1.2, WB1-A-R3.1
- new net WB1-A-OUT: AMP-1.OUTA, WB1-A-R3.2, WB1-A-R5.1, WB2-A-R3.2, WB2-A-R5.1, WB4-A-R3.2, WB4-A-R5.1, WB6-A-R3.2, WB6-A-R5.1
- new net WB1-A-POS: AMP-1.+INA, WB1-A-R2.2, WB1-A-R4.2
- new net WB10-A-NEG: AMP-3.-INB, WB10-A-R1.2, WB10-A-R3.1
- new net WB10-A-OUT: AMP-3.OUTB, WB10-A-R3.2, WB10-A-R5.1
- new net WB10-A-POS: AMP-3.+INB, WB10-A-R2.2, WB10-A-R4.2
- new net WB11-A-NEG: AMP-3.-INC, WB11-A-R1.2, WB11-A-R3.1
- new net WB11-A-OUT: AMP-3.OUTC, WB11-A-R3.2, WB11-A-R5.1
- new net WB11-A-POS: AMP-3.+INC, WB11-A-R2.2, WB11-A-R4.2
- new net WB12-A-NEG: AMP-3.-IND, WB12-A-R1.2, WB12-A-R3.1
- new net WB12-A-OUT: AMP-3.OUTD, WB12-A-R3.2, WB12-A-R5.1
- new net WB12-A-POS: WB12-A-R2.2, WB12-A-R4.2
- new net WB124-A-POS: AMP-3.+IND
- new net WB2-A-NEG: AMP-1.-INB, WB2-A-R1.2, WB2-A-R3.1
- new net WB2-A-OUT: AMP-1.OUTB
- new net WB2-A-POS: AMP-1.+INB, WB2-A-R2.2, WB2-A-R4.2
- new net WB3-A-NEG: AMP-1.-INC, WB3-A-R1.2, WB3-A-R3.1
- new net WB3-A-OUT: AMP-1.OUTC, WB3-A-R3.2, WB3-A-R5.1
- new net WB3-A-POS: AMP-1.+INC, WB3-A-R2.2, WB3-A-R4.2
- new net WB4-A-NEG: AMP-1.-IND, WB4-A-R1.2, WB4-A-R3.1
- new net WB4-A-OUT: AMP-1.OUTD
- new net WB4-A-POS: AMP-1.+IND, WB4-A-R2.2, WB4-A-R4.2
- new net WB5-A-NEG: AMP-2.-INA, WB5-A-R1.2, WB5-A-R3.1
- new net WB5-A-OUT: AMP-2.OUTA, WB5-A-R3.2, WB5-A-R5.1
- new net WB5-A-POS: AMP-2.+INA, WB5-A-R2.2, WB5-A-R4.2
- new net WB6-A-NEG: AMP-2.-INB, WB6-A-R1.2, WB6-A-R3.1
- new net WB6-A-OUT: AMP-2.OUTB
- new net WB6-A-POS: AMP-2.+INB, WB6-A-R2.2, WB6-A-R4.2
- new net WB7-A-NEG: AMP-2.-INC, WB7-A-R1.2, WB7-A-R3.1
- new net WB7-A-OUT: AMP-2.OUTC, WB7-A-R3.2, WB7-A-R5.1
- new net WB7-A-POS: AMP-2.+INC, WB7-A-R2.2, WB7-A-R4.2
- new net WB8-A-NEG: AMP-2.-IND, WB8-A-R1.2, WB8-A-R3.1
- new net WB8-A-OUT: AMP-2.OUTD, WB8-A-R3.2, WB8-A-R5.1
- new net WB8-A-POS: AMP-2.+IND, WB8-A-R2.2, WB8-A-R4.2
- new net WB9-A-NEG: AMP-3.-INA, WB9-A-R1.2, WB9-A-R3.1
- new net WB9-A-OUT: AMP-3.OUTA, WB9-A-R3.2, WB9-A-R5.1
- new net WB9-A-POS: AMP-3.+INA, WB9-A-R2.2, WB9-A-R4.2
- net +5V: now also 5VSUP-BYP.1, ADC-1.VDD, ADC-BYP.1, ATMEGA328-BYP.2, ATMEGA328.AREF, ATMEGA328.AVCC, ATMEGA328.VCC@4, ATMEGA328.VCC@6, CAL-1.GA, CAL-10.GA, CAL-11.GA, CAL-12.GA, CAL-13.GA, CAL-14.GA, CAL-15.GA, CAL-16.GA, CAL-2.GA, CAL-3.GA, CAL-4.GA, CAL-5.GA, CAL-6.GA, CAL-7.GA, CAL-8.GA, CAL-9.GA, ICSP.2, LSHIFT-1.VCCB, LSHIFT-2.VCCB, LSHIFT1-BYP-2.1, LSHIFT2-BYP-2.1, RESET-PULLUP.2, SHREG-BYP.1, SHREGP.VCC; no longer D1.GA, IC3P.VCC, U3.VDD, U4.AREF, U4.AVCC, U4.PC6(/RESET), U4.VCC@4, U4.VCC@6, U5.VCCB
- net GND: now also -3VSUP-BYP.1, -3VSUP.IN, 3VSUP-BYP.2, 5VSUP-BYP.2, ADC-1.GND, ADC-BYP.2, AMP-1.NC, AMP-1.NC_2, AMP-2.NC, AMP-2.NC_2, AMP-3.NC, AMP-3.NC_2, ATMEGA328-BYP.1, ATMEGA328.AGND, ATMEGA328.GND@3, ATMEGA328.GND@5, CAL-1-R1.1, CAL-10-R1.1, CAL-11-R1.1, CAL-12-R1.1, CAL-13-R1.1, CAL-14-R1.1, CAL-15-R1.1, CAL-16-R1.1, CAL-2-R1.1, CAL-3-R1.1, CAL-4-R1.1, CAL-5-R1.1, CAL-6-R1.1, CAL-7-R1.1, CAL-8-R1.1, CAL-9-R1.1, CRYSTAL-C1.1, CRYSTAL-C2.1, ICSP.6, INPUT-BYP.2, LSHIFT-1.GND, LSHIFT-2.GND, LSHIFT1-BYP-1.2, LSHIFT1-BYP-2.2, LSHIFT2-BYP-1.2, LSHIFT2-BYP-2.2, POT-1.DGND, POT-1.VSS, POT-2.DGND, POT-2.VSS, POT-3.DGND, POT-3.VSS, POT1-BYP.2, POT2-BYP.2, POT3-BYP.2, SD-BYP.2, SD-SOCKET.SH@1, SD-SOCKET.SH@2, SD-SOCKET.VSS1, SD-SOCKET.VSS2, SHREG-BYP.2, SHREGP.GND, WB1-A-C1.2, WB1-A-R4.1, WB1-R1.1, WB1-R2.1, WB10-A-C1.2, WB10-A-R4.1, WB10-R1.1, WB10-R2.1, WB11-A-C1.2, WB11-A-R4.1, WB11-R1.1, WB11-R2.1, WB12-A-C1.2, WB12-A-R4.1, WB12-R1.1, WB12-R2.1, WB2-A-C1.2, WB2-A-R4.1, WB2-R1.1, WB2-R2.1, WB3-A-C1.2, WB3-A-R4.1, WB3-R1.1, WB3-R2.1, WB4-A-C1.2, WB4-A-R4.1, WB4-R1.1, WB4-R2.1, WB5-A-C1.2, WB5-A-R4.1, WB5-R1.1, WB5-R2.1, WB6-A-C1.2, WB6-A-R4.1, WB6-R1.1, WB6-R2.1, WB7-A-C1.2, WB7-A-R4.1, WB7-R1.1, WB7-R2.1, WB8-A-C1.2, WB8-A-R4.1, WB8-R1.1, WB8-R2.1, WB9-A-C1.2, WB9-A-R4.1, WB9-R1.1, WB9-R2.1; no longer C1.1, C2.2, C4.1, C5.1, IC3P.GND, J1.SH@1, J1.SH@2, J1.VSS1, J1.VSS2, R1.1, R16.1, R2.1, U1.V-, U3.GND, U4.AGND, U4.GND@3, U4.GND@5, U5.GND
- net N$1: now also -3VSUP-D1.A, -3VSUP-R3.2; no longer R2.2, R3.1, R5.1, U2.B0
- net N$13: now also LSHIFT-2.A3, SD-SOCKET.CD/DAT3; no longer J1.CD/DAT3, U5.A3
- net N$15: now also LSHIFT-2.A1, SD-SOCKET.WP; no longer J1.WP, U5.A1
- net N$17: now also LSHIFT-2.A2, SD-SOCKET.CD; no longer J1.CD, U5.A2
- net N$18: now also LSHIFT-2.A4, SD-SOCKET.CMD; no longer J1.CMD, U5.A4
- net N$19: now also ATMEGA328.PB6(XTAL1/TOSC1), CRYSTAL-C1.2, CRYSTAL.2; no longer C4.2, Q1.2, U4.PB6(XTAL1/TOSC1)
- net N$2: now also -3VSUP-R1.1, -3VSUP-R2.2, -3VSUP.ADJ; no longer R1.2, R6.1, X1-2.1
- net N$20: now also ATMEGA328.PB7(XTAL2/TOSC2), CRYSTAL-C2.2, CRYSTAL.1; no longer C5.2, Q1.1, U4.PB7(XTAL2/TOSC2)
- net N$21: now also LSHIFT-1.A1, SD-SOCKET.CLK; no longer J1.CLK, U5.A5
- net N$22: now also LSHIFT-1.A2, SD-SOCKET.DAT2; no longer J1.DAT2, U5.A6
- net N$23: now also LSHIFT-1.A3, SD-SOCKET.DAT1; no longer J1.DAT1, U5.A7
- net N$24: now also LSHIFT-1.A4, SD-SOCKET.DAT0; no longer J1.DAT0, U5.A8
- net N$25: now also CAL-1-R1.2, CAL-1.RC; no longer D1.RC, R16.2
- net N$26: now also CAL-1-R2.2, CAL-1.GC; no longer D1.GC, R17.2
- net N$27: now also CAL-1-R2.1, CAL-1.RA, SHREGA.P0; no longer D1.RA, IC3A.P0, R17.1
- net N$28: now also ATMEGA328.PD4(XCK/T0), LSHIFT-2.B1; no longer U4.PB5(SCK), U5.B1
- net N$29: now also ATMEGA328.PD1(TXD), LSHIFT-2.B2; no longer U4.PB4(MISO), U5.B2
- net N$30: now also ATMEGA328.PD0(RXD), LSHIFT-2.B3; no longer U4.PB3(MOSI/OC2), U5.B3
- net N$31: now also ATMEGA328.PB2(SS/OC1B), LSHIFT-2.B4; no longer U4.PB2(SS/OC1B), U5.B4
- net N$32: now also ATMEGA328.PB1(OC1A), LSHIFT-1.B1; no longer U4.PB1(OC1A), U5.B5
- net N$33: now also ATMEGA328.PB0(ICP), LSHIFT-1.B2; no longer U4.PB0(ICP), U5.B6
- net N$34: now also ATMEGA328.PD7(AIN1), LSHIFT-1.B3; no longer U4.PD7(AIN1), U5.B7
- net N$35: now also ATMEGA328.PD6(AIN0), LSHIFT-1.B4; no longer U4.PD6(AIN0), U5.B8
- net N$36: now also ATMEGA328.PC3(ADC3), SHREGA.SER/Q15; no longer IC3A.SER/Q15, U4.PC3(ADC3)
- net N$37: now also ATMEGA328.PC0(ADC0), SHREGA.CLK; no longer IC3A.CLK, U4.PC0(ADC0)
- net N$38: now also ATMEGA328.PC1(ADC1), SHREGA.MOD; no longer IC3A.MOD, U4.PC1(ADC1)
- net N$39: now also ATMEGA328.PC2(ADC2), SHREGA.R/!W; no longer IC3A.R/!W, U4.PC2(ADC2)
- net N$40: now also ATMEGA328.ADC6, SHREGA.CS; no longer IC3A.CS, U4.ADC6
- net N$5: now also ATMEGA328.ADC7, POT-WP-R1.2; no longer R4.2, U2.W0
- net VCC: now also INPUT-BYP.1
Other:
- note added: "NC"
- note removed: "AMPLIFIER"
- note removed: "AMPLIFIER CIRCUIT"
- moved on the sheet: X1-1, X1-2, X1-3, X1-4, X1-5, X1-6
