File: 12T_GAUGE_INPUT.sch (EAGLE design)
At the start: 102 parts, among them J1 MICRO-SD_CARD_SOCKET, P1_WP_PULLUP 10k, P2_WP_PULLUP 10k, P3_WP_PULLUP 10k, U15 WS2812

Commit message: Fixed wheatstone bridges
forgot a resistor on bridge
Parts:
- removed 3V-R1: 240, rcl:R-US_R1206
- removed 3V-R2: 390, rcl:R-US_R1206
- removed 3V3-DCPL: 10uF, rcl:C-USC1206
- removed 3VREG: V_REG_317SMD, SparkFun-IC-Power:V_REG_317SMD
- added B10R3, B11R3, B12R3, B1R3, B2R3, B3R3, B4R3, B5R3, B6R3, B7R3, B8R3, B9R3: 370, rcl:R-US_R1206
- added RTC_DCPL: 10uF, rcl:C-USC1206
- renumbered U15 to CAL12
Connections:
- removed net +3V3: 3V-R1.2, 3V3-DCPL.1, 3VREG.OUT
- removed net N$8: 3V-R1.1, 3V-R2.2, 3VREG.ADJ
- net +12V: no longer 3VREG.IN
- net +5V: now also RTC_DCPL.1
- net B1-_P1W0: now also B1R3.1
- net B10-_P3W1: now also B10R3.1
- net B11-_P3W2: now also B11R3.1
- net B12-_P3W3: now also B12R3.1
- net B2-_P1W1: now also B2R3.1
- net B3-_P1W2: now also B3R3.1
- net B4-_P1W3: now also B4R3.1
- net B5-_P2W0: now also B5R3.1
- net B6-_P2W1: now also B6R3.1
- net B7-_P2W2: now also B7R3.1
- net B8-_P2W3: now also B8R3.1
- net B9-_P3W0: now also B9R3.1
- net GND: now also RTC_DCPL.2; no longer 3V-R2.1, 3V3-DCPL.2
- net V+: now also B10R3.2, B11R3.2, B12R3.2, B1R3.2, B2R3.2, B3R3.2, B4R3.2, B5R3.2, B6R3.2, B7R3.2, B8R3.2, B9R3.2

Commit message: Readability, and made board smaller (again)
Schematic: Moved things around to make it more easily read

Board: Moved things around to shrink the board and increase the ground plane area
Parts:
- removed 5VREG, GAUGE_REG: V_REG_317SMD, SparkFun-IC-Power:V_REG_317SMD
- removed J1: MICRO-SD_CARD_SOCKET, SparkFun-Connectors:MICRO-SD_CARD_SOCKET
- removed MEGA_RESET_PULLUP, SCL_PULLUP, SDA_PULLUP: 10k, rcl:R-US_R1206
- removed PWR-DCPL-AGND, PWR-DCPL-GND, VREF-DCPL: 10uF, rcl:C-USC1206
- removed VREF-R2: 100, rcl:R-US_R1206
- added +5V, GAUGE: V_REG_317SMD, SparkFun-IC-Power:V_REG_317SMD
- added MEGA_RST, SCL_PULL, SDA_PULL: 10k, rcl:R-US_R1206
- added PWR-DCPL1, PWR-DCPL2, VREF_C1: 10uF, rcl:C-USC1206
- added SD_SLOT: MICRO-SD_CARD_SOCKET, SparkFun-Connectors:MICRO-SD_CARD_SOCKET
- added VREF_R2: 100, rcl:R-US_R1206
- CAL1, CAL10, CAL11, CAL12, CAL2, CAL3, CAL4, CAL5, CAL6, CAL7, CAL8, CAL9: value WS2812 -> WS2812"
- renumbered P1_WP_PULLUP to P1_WP, P2_WP_PULLUP to P2_WP, P3_WP_PULLUP to P3_WP
Connections:
- net N$2 renamed MEGA_XTAL1
- net N$21 renamed +3V
- net N$3 renamed MEGA_XTAL2
- removed net AGND: ADS1-DCPL1.2, ADS1B.AGND, ADS1B.VREFN, ADS2-DCPL1.2, ADS2B.AGND, ADS3-DCPL1.2, ADS3B.AGND, B1-R1.1, B10-R1.1, B11-R1.1, B12-R1.1, B2-R1.1, B3-R1.1, B4-R1.1, B5-R1.1, B6-R1.1, B7-R1.1, B8-R1.1, B9-R1.1, GAUGE1-2.1, GAUGE10-2.1, GAUGE11-2.1, GAUGE12-2.1, GAUGE2-2.1, GAUGE3-2.1, GAUGE4-2.1, GAUGE5-2.1, GAUGE6-2.1, GAUGE7-2.1, GAUGE8-2.1, GAUGE9-2.1, PWR-DCPL-AGND.2, PWR-IN-3.1, VREF-DCPL.2, VREF-R2.1
- net +12V: now also +5V.IN, GAUGE.IN, PWR-DCPL1.1, PWR-DCPL2.1; no longer 5VREG.IN, GAUGE_REG.IN, PWR-DCPL-AGND.1, PWR-DCPL-GND.1
- net +5V: now also +5V.OUT, MEGA_RST.2, SCL_PULL.2, SDA_PULL.2, SD_SLOT.VCC; no longer 5VREG.OUT, J1.VCC, MEGA_RESET_PULLUP.2, SCL_PULLUP.2, SDA_PULLUP.2
- net GND: now also ADS1-DCPL1.2, ADS1B.AGND, ADS1B.VREFN, ADS2-DCPL1.2, ADS2B.AGND, ADS3-DCPL1.2, ADS3B.AGND, B1-R1.1, B10-R1.1, B11-R1.1, B12-R1.1, B2-R1.1, B3-R1.1, B4-R1.1, B5-R1.1, B6-R1.1, B7-R1.1, B8-R1.1, B9-R1.1, GAUGE1-2.1, GAUGE10-2.1, GAUGE11-2.1, GAUGE12-2.1, GAUGE2-2.1, GAUGE3-2.1, GAUGE4-2.1, GAUGE5-2.1, GAUGE6-2.1, GAUGE7-2.1, GAUGE8-2.1, GAUGE9-2.1, PWR-DCPL1.2, PWR-DCPL2.2, PWR-IN-3.1, SD_SLOT.CD1, SD_SLOT.CD2, SD_SLOT.GND, SD_SLOT.SHIELD@1, SD_SLOT.SHIELD@3, VREF_C1.2, VREF_R2.1; no longer J1.CD1, J1.CD2, J1.GND, J1.SHIELD@1, J1.SHIELD@3, PWR-DCPL-GND.2
- net MISO: now also SD_SLOT.DO; no longer J1.DO
- net MOSI: now also SD_SLOT.DI; no longer J1.DI
- net N$11: now also GAUGE.ADJ; no longer GAUGE_REG.ADJ
- net N$5: now also +5V.ADJ; no longer 5VREG.ADJ
- net RESET: now also MEGA_RST.1; no longer MEGA_RESET_PULLUP.1
- net SCK: now also SD_SLOT.SCK; no longer J1.SCK
- net SCL: now also SCL_PULL.1; no longer SCL_PULLUP.1
- net SDA: now also SDA_PULL.1; no longer SDA_PULLUP.1
- net SD_CS: now also SD_SLOT.!CS; no longer J1.!CS
- net V+: now also GAUGE.OUT; no longer GAUGE_REG.OUT
- net VREF: now also VREF_C1.1, VREF_R2.2; no longer VREF-DCPL.1, VREF-R2.2
Other:
- moved on the sheet: 5V-DCPL, 5V-R1, 5V-R2, 6V-R1, 6V-R2, ADS1-DCPL1, ADS1-DCPL2, ADS1A, ADS1B, ADS2-DCPL1, ADS2-DCPL2, ADS2A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
