File: Racing_Sensors_Connector/CanBusArduino.sch (EAGLE design)
At the start: 25 parts, among them U2 SPARKFUN_USD-SOCKETSMD, U3 AT90CAN128-16AI

Commit message: Teensy shield version
Parts:
- removed ADC0/1, ADC2/3, ADC4/5, ADC6/7, I2C, TX/RX: (no value), SparkFun-Connectors:CONN_02POLAR
- removed BYP2: 0.1uF, SparkFun-Capacitors:0.1UF-0603-25V-(+80/-20%)
- removed COSC1, COSC2: 22pF, SparkFun-Capacitors:22PF-0603-50V-5%
- removed ISP: (no value), SparkFun-Connectors:CONN_03X22X3_SILK_MALE_PTH
- removed OSC: 16MHz, SparkFun-Clocks:CRYSTALPTH-HC49US
- removed PRGM: (no value), SparkFun-Connectors:CONN_03
- removed RST_PULLUP: 10k, SparkFun-Resistors:10KOHM-0603-1/10W-1%
- removed U3: AT90CAN128-16AI, _hhn_at90can32_64_128_v2:AT90CAN128-16AI
- added BT1: (no value), SparkFun-Batteries:BATTERY-20MM_SMD_4LEGS
- added TEENSY: TEENSY_3.1-3.2_ALL_PINS, Teensy_3_and_LC_Series_Boards_v1.4:TEENSY_3.1-3.2_ALL_PINS
- renumbered CAP_CANH to CCANH, CAP_CANL to CCANL, R2 to RCANL, R3 to RCANH
Connections:
- removed net A4: ADC4/5.2, U3.PF4(ADC4/TCK)
- removed net A5: ADC4/5.1, U3.PF5(ADC5/TMS)
- removed net OSC1: COSC1.1, OSC.2, U3.XTAL1
- removed net OSC2: COSC2.1, OSC.1, U3.XTAL2
- removed net RESET: ISP.5, PRGM.3, RST_PULLUP.1, U3.!RESET
- removed net RX: PRGM.1, U3.(RXD0/PDI)PE0
- removed net TX: PRGM.2, U3.(TXD0/PDO)PE1
- new net 3.3V: SD_PULLUP.2, TEENSY.3.3V, U2.VCC
- new net 3V: BT1.+, TEENSY.VBAT
- new net A8: TEENSY.22/A8/T/PWM
- new net A9: TEENSY.23/A9/T/PWM
- net A0: now also TEENSY.14/A0; no longer ADC0/1.2, U3.PF0(ADC0)
- net A1: now also TEENSY.15/A1/T; no longer ADC0/1.1, U3.PF1(ADC1)
- net A2: now also TEENSY.16/A2/T; no longer ADC2/3.2, U3.PF2(ADC2)
- net A3: now also TEENSY.17/A3/T; no longer ADC2/3.1, U3.PF3(ADC3)
- net A6: now also TEENSY.20/A6/PWM; no longer ADC6/7.2, U3.PF6(ADC6/TDO)
- net A7: now also TEENSY.21/A7/PWM; no longer ADC6/7.1, U3.PF7(ADC7/TDI)
- net CAN_RXD: now also TEENSY.4/CAN-RX/PWM; no longer U3.(RXCAN/T1)PD6
- net CAN_STBY: now also TEENSY.5/PWM; no longer U3.(AD5)PA5
- net CAN_TXD: now also TEENSY.3/CAN-TX/PWM; no longer U3.(TXCAN/XCK1)PD5
- net GND: now also BT1.-, TEENSY.AGND, TEENSY.GND; no longer BYP2.2, COSC1.2, COSC2.2, ISP.6, U3.GND@1, U3.GND@2, U3.GND@3
- net MISO: now also TEENSY.12/MISO; no longer ISP.1, U3.(MISO)PB3
- net MOSI: now also TEENSY.11/MOSI; no longer ISP.4, U3.(MOSI)PB2
- net RX1: now also TEENSY.0/RX1/T; no longer TX/RX.2, U3.(RXD1/INT2)PD2
- net SCK: now also TEENSY.13/SCK/LED; no longer ISP.3, U3.(SCK)PB1
- net SCL: now also TEENSY.19/A5/T/SCL0; no longer I2C.2, U3.(SCL/INT0)PD0
- net SDA: now also TEENSY.18/A4/T/SDA0; no longer I2C.1, U3.(SDA/INT1)PD1
- net SD_CD: now also TEENSY.7/RX3; no longer U3.(AD7)PA7
- net SD_CS: now also TEENSY.6/PWM; no longer U3.(AD6)PA6
- net TX1: now also TEENSY.1/TX1/T; no longer TX/RX.1, U3.(TXD1/INT3)PD3
- net VCC: now also TEENSY.VIN; no longer BYP2.1, ISP.2, RST_PULLUP.2, SD_PULLUP.2, U2.VCC, U3.AVCC, U3.VCC@1, U3.VCC@2
Other:
- note removed: "Backup Arduino programmer"
- note removed: "Programming ISP header for Atmel ICE"
